File: PCM5102A_DAC.kicad_sch (KiCad schematic)
At the start: 35 parts, among them U1 AP7365-33YG, U3 PCM5102A, U4 AP7365-33YG

Commit message: first
Parts:
- removed A3V3DAC1, A3V3DAC2, AGNDDAC1, D3V3DAC1, DAC_OUT_L1, DAC_OUT_R1, GND3: TP, TestPoint:TestPoint_Pad_1.0x1.0mm, symbol Connector:TestPoint
- removed JP1, JP2, JP3: SolderJumper_2_Bridged, Jumper:SolderJumper-2_P1.3mm_Bridged_Pad1.0x1.5mm, symbol Jumper:SolderJumper_2_Bridged
Connections:
- net GND: now also U3.10 (DEMP), U3.11 (FLT), U3.16 (FMT)
Other:
- note removed: "test points"
