File: TeensyHapticAudioPlayer.kicad_pcb (KiCad board)
At the start: 2 copper layers, 57 parts, among them J1 Conn_01x04, J2 AudioJack3, J3 Micro_SD_Card, U1 Teensy4.0, U2 AP7365-33YG, U3 AP7365-33YG, U4 PCM5102A

Commit message: first
Parts:
- removed A3V3DAC1, A3V3DAC2, AGNDDAC1, D3V3DAC1, DAC_OUT_L1, DAC_OUT_R1, GND1: TP, TestPoint:TestPoint_Pad_1.0x1.0mm
- removed JP2, JP3, JP4: SolderJumper_2_Bridged, Jumper:SolderJumper-2_P1.3mm_Bridged_Pad1.0x1.5mm
- removed POWER ON1: LED, LED_SMD:LED_0603_1608Metric
- removed R1: 10K, Resistor_SMD:R_0603_1608Metric_Pad0.98x0.95mm_HandSolder
- added 3vpins1: Conn_01x12, Connector_PinSocket_2.54mm:PinSocket_1x12_P2.54mm_Vertical, F.Cu at (53.8, 18.5)
- added AGND_BRIDGE2: AGND_BRIDGE, Jumper:SolderJumper-2_P1.3mm_Bridged_Pad1.0x1.5mm, F.Cu at (75.5, 47.7)
- added C20: 10uf, Capacitor_SMD:CP_Elec_5x5.7, F.Cu at (60.7, 32.9)
- added C21: 1uf, Capacitor_SMD:C_0603_1608Metric, F.Cu at (67.4, 22.4)
- added C22: 0.1uf, Capacitor_SMD:C_0603_1608Metric_Pad1.08x0.95mm_HandSolder, F.Cu at (66.4, 32.9)
- added C23: 1uf, Capacitor_SMD:C_0603_1608Metric, F.Cu at (61.1, 25.1)
- added C24: 1uf, Capacitor_SMD:C_0603_1608Metric, F.Cu at (65.2, 29.4)
- added GNDpins1: Conn_01x12, Connector_PinSocket_2.54mm:PinSocket_1x12_P2.54mm_Vertical, F.Cu at (53.8, 23.1)
- added J4: Conn_01x04_Pin, Connector_PinSocket_2.54mm:PinSocket_1x04_P2.54mm_Vertical, F.Cu at (75.0, 64.3)
- added JP6: SolderJumper_3_Bridged12, Jumper:SolderJumper-3_P1.3mm_Bridged12_Pad1.0x1.5mm, F.Cu at (89.4, 39.4)
- added R12: 10k, Resistor_SMD:R_0603_1608Metric_Pad0.98x0.95mm_HandSolder, F.Cu at (63.3, 19.7)
- added R13: 10k, Resistor_SMD:R_0603_1608Metric_Pad0.98x0.95mm_HandSolder, F.Cu at (63.3, 22.3)
- added R14: 10k, Resistor_SMD:R_0603_1608Metric_Pad0.98x0.95mm_HandSolder, F.Cu at (81.7, 61.4)
- added R15: 10k, Resistor_SMD:R_0603_1608Metric_Pad0.98x0.95mm_HandSolder, F.Cu at (81.7, 59.7)
- added STEMMA_QT_I2C1: JST_SH_SM04, Connector_JST:JST_SH_SM04B-SRSS-TB_1x04-1MP_P1.00mm_Horizontal, F.Cu at (90.2, 63.2)
- added U5: DRV2605LDGS, Package_SO:VSSOP-10_3x3mm_P0.5mm, F.Cu at (66.3, 26.2)
- added VIBMTR1: VIBMTR, TerminalBlock:TerminalBlock_bornier-2_P5.08mm, F.Cu at (78.3, 19.5)
- added extra_gpio1: Conn_01x12, Connector_PinSocket_2.54mm:PinSocket_1x12_P2.54mm_Vertical, F.Cu at (53.8, 27.7)
- moved C3 137.5 mm to (58.3, 49.1)
- moved C4 131.2 mm to (64.9, 41.0), turned to 90 degrees
- moved C2 131.1 mm to (60.0, 42.9)
- moved C7 130.2 mm to (60.4, 40.1), turned to 90 degrees
- moved U3 129.9 mm to (60.7, 54.0), turned to -90 degrees
- moved C5 129.3 mm to (67.1, 56.9), turned to -90 degrees
- moved C8 125.2 mm to (62.5, 58.8), turned to -90 degrees
- moved U2 123.6 mm to (63.0, 47.7), turned to -90 degrees
- moved C6 120.6 mm to (71.0, 41.0), turned to 90 degrees
- moved C9 117.9 mm to (77.4, 44.0), turned to -90 degrees
- moved C10 104.8 mm to (76.9, 40.7), turned to -90 degrees
- moved C13 103.6 mm to (75.3, 40.9), turned to -90 degrees
- moved C11 101.0 mm to (77.8, 35.5)
- moved C12 98.5 mm to (77.9, 37.5)
- moved U4 95.4 mm to (82.0, 44.2), turned to -90 degrees
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Connections:
- J1 pad 3: /DAC_OUT_R -> /audio_out_chan2
- J2 pad R: /DAC_OUT_R -> /audio_out_chan2
- U1 pad 1: unconnected-(U1-GND-Pad1) -> GND
- U1 pad 10: unconnected-(U1-8_TX2_IN1-Pad10) -> /gp8
- U1 pad 11: unconnected-(U1-9_OUT1C-Pad11) -> /gp9
- U1 pad 12: unconnected-(U1-10_CS_MQSR-Pad12) -> /SD_CS
- U1 pad 13: unconnected-(U1-11_MOSI_CTX1-Pad13) -> /SD_MOSI
- U1 pad 14: unconnected-(U1-12_MISO_MQSL-Pad14) -> /SD_MISO
- U1 pad 16: unconnected-(U1-3V3-Pad16) -> +3.3V
- U1 pad 17: unconnected-(U1-GND-Pad17) -> GND
- U1 pad 2: unconnected-(U1-0_RX1_CRX2_CS1-Pad2) -> /gp0
- U1 pad 20: unconnected-(U1-13_SCK_CRX1_LED-Pad20) -> /SD_SCK
- U1 pad 21: unconnected-(U1-14_A0_TX3_SPDIF_OUT-Pad21) -> /gp14
- U1 pad 22: unconnected-(U1-15_A1_RX3_SPDIF_IN-Pad22) -> /gp15
- U1 pad 23: unconnected-(U1-16_A2_RX4_SCL1-Pad23) -> /I2C1_SCL
- U1 pad 24: unconnected-(U1-17_A3_TX4_SDA1-Pad24) -> /I2C1_SDA
- U1 pad 25: unconnected-(U1-18_A4_SDA0-Pad25) -> /I2C0_SDA
- U1 pad 26: unconnected-(U1-19_A5_SCL0-Pad26) -> /I2C0_SCL
- U1 pad 29: unconnected-(U1-22_A8_CTX1-Pad29) -> /gp22
- U1 pad 3: unconnected-(U1-1_TX1_CTX2_MISO1-Pad3) -> /gp1
- U1 pad 30: unconnected-(U1-23_A9_CRX1_MCLK1-Pad30) -> /gp23
- U1 pad 32: unconnected-(U1-GND-Pad32) -> GND
- U1 pad 33: unconnected-(U1-VIN-Pad33) -> +5V
- U1 pad 4: unconnected-(U1-2_OUT2-Pad4) -> /gp2
- U1 pad 5: unconnected-(U1-3_LRCLK2-Pad5) -> /gp3
- U1 pad 6: unconnected-(U1-4_BCLK2-Pad6) -> /gp4
- U1 pad 7: unconnected-(U1-5_IN2-Pad7) -> /NEOPIXEL
- U1 pad 8: unconnected-(U1-6_OUT1D-Pad8) -> /gp6
- U4 pad 10: Net-(JP2-B) -> GND
- U4 pad 11: Net-(JP3-B) -> GND
- U4 pad 16: Net-(JP4-B) -> GND
Routing:
- net GND: track 0.00 -> 334.9 mm, vias 0 -> 15
- net +3.3V: track 0.00 -> 232.8 mm, vias 0 -> 6
- net +5V: track 0.00 -> 104.7 mm, vias 0 -> 5
- net /AGND: track 0.00 -> 88.6 mm, vias 0 -> 8
- net /I2C1_SCL: track 0.00 -> 88.2 mm
- net /I2C1_SDA: track 0.00 -> 76.4 mm, vias 0 -> 2
- net /DAC_LRCK: track 0.00 -> 62.4 mm, vias 0 -> 2
- net /DAC_BCK: track 0.00 -> 59.1 mm, vias 0 -> 2
- net /gp1: track 0.00 -> 57.9 mm, vias 0 -> 1
- net /PCM5102A DAC/3V3A: track 0.00 -> 53.6 mm, vias 0 -> 3
- net /gp0: track 0.00 -> 53.2 mm, vias 0 -> 3
- net /gp2: track 0.00 -> 52.4 mm, vias 0 -> 1
- net /DAC_DIN: track 0.00 -> 52.4 mm, vias 0 -> 1
- net /gp3: track 0.00 -> 45.6 mm, vias 0 -> 1
- net /gp9: track 0.00 -> 41.9 mm, vias 0 -> 3
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- added copper zone on B.Cu, net /AGND
- added copper zone on F.Cu, net /AGND
- added copper zone on B.Cu, net GND
- added copper zone on F.Cu, net GND
Other:
- board outline added: 79.9 x 53.5 mm
- board text added: "0 1 2 3 4 6 8 9 14 15 22 23"
- board text added: "3V"
- board text added: "CONNECTIONS DAC: DIN->7 LRCK->20 BCK->21 SD: CS->10 MOSI->11 MISO->12 Neopixel->5 DRV2605 via i2c0: SDA->18 SCL->19 StemmaQT via i2c1: SCL->16 SDA->17"
- board text added: "G"
- board text added: "G 3V SDA SCL"
- board text added: "G M 3V"
- board text added: "G-AG"
- board text added: "GPIO"
- board text added: "L"
- board text added: "P 3v G"
- board text added: "R"
- board text added: "SD"
- board text added: "Teensy Haptic Audio Board by Mads Kjeldgaard for hyaline.systems 2025 ⊂(◉‿◉)つ https://hyaline.systems"
- board text added: "VIB -+"
- board text added: "cut to mute ->"
- board text added: "drv to dac_l->"
- board text added: "i2c1"
- board text added: "teensy 4.0 goes here"
