File: TeensyHapticAudioPlayer.kicad_sch (KiCad schematic)
At the start: 15 parts, among them J1 Conn_01x04, J2 AudioJack3, U1 Teensy4.0

Commit message: first
Parts:
- removed POWER ON1: LED, LED_SMD:LED_0603_1608Metric, symbol Device:LED
- removed R1: 10K, Resistor_SMD:R_0603_1608Metric_Pad0.98x0.95mm_HandSolder, symbol Device:R
- added 3vpins1, GNDpins1, extra_gpio1: Conn_01x12, Connector_PinSocket_2.54mm:PinSocket_1x12_P2.54mm_Vertical, symbol Connector_Generic:Conn_01x12
- added AGND_BRIDGE2: AGND_BRIDGE, Jumper:SolderJumper-2_P1.3mm_Bridged_Pad1.0x1.5mm, symbol Jumper:SolderJumper_2_Bridged
- added C24: 1uf, Capacitor_SMD:C_0603_1608Metric, symbol Device:C
- added J4: Conn_01x04_Pin, Connector_PinSocket_2.54mm:PinSocket_1x04_P2.54mm_Vertical, symbol Connector:Conn_01x04_Pin
- added JP6: SolderJumper_3_Bridged12, Jumper:SolderJumper-3_P1.3mm_Bridged12_Pad1.0x1.5mm, symbol Jumper:SolderJumper_3_Bridged12
- added R14, R15: 10k, Resistor_SMD:R_0603_1608Metric_Pad0.98x0.95mm_HandSolder, symbol Device:R
- added STEMMA_QT_I2C1: JST_SH_SM04, Connector_JST:JST_SH_SM04B-SRSS-TB_1x04-1MP_P1.00mm_Horizontal, symbol Connector:Conn_01x04_Pin
Connections:
- net +3.3V: now also U1.16 (3V3), 3vpins1.1 (Pin_1), 3vpins1.10 (Pin_10), 3vpins1.11 (Pin_11), 3vpins1.12 (Pin_12), 3vpins1.2 (Pin_2), 3vpins1.3 (Pin_3), 3vpins1.4 (Pin_4), 3vpins1.5 (Pin_5), 3vpins1.6 (Pin_6), 3vpins1.7 (Pin_7), 3vpins1.8 (Pin_8), 3vpins1.9 (Pin_9), J4.2 (Pin_2), R14.1, R15.2, STEMMA_QT_I2C1.2 (Pin_2)
- net +5V: now also U1.33 (VIN)
- net DAC_OUT_L: now also JP6.1 (A)
- net DAC_OUT_R: now also AGND_BRIDGE2.1 (A), JP6.3 (B); no longer J1.3 (Pin_3), J2.R
- net GND: now also U1.1 (GND), U1.17 (GND), U1.32 (GND), GNDpins1.1 (Pin_1), GNDpins1.10 (Pin_10), GNDpins1.11 (Pin_11), GNDpins1.12 (Pin_12), GNDpins1.2 (Pin_2), GNDpins1.3 (Pin_3), GNDpins1.4 (Pin_4), GNDpins1.5 (Pin_5), GNDpins1.6 (Pin_6), GNDpins1.7 (Pin_7), GNDpins1.8 (Pin_8), GNDpins1.9 (Pin_9), J4.1 (Pin_1), STEMMA_QT_I2C1.1 (Pin_1)
- net NEOPIXEL: now also U1.7 (5_IN2)
- net SD_CS: now also U1.12 (10_CS_MQSR)
- net SD_MISO: now also U1.14 (12_MISO_MQSL)
- net SD_MOSI: now also U1.13 (11_MOSI_CTX1)
- net SD_SCK: now also U1.20 (13_SCK_CRX1_LED)
- net gp8: now reaches U1.10 (8_TX2_IN1)
- net gp8: now also extra_gpio1.7 (Pin_7)
- net gp9: now reaches U1.11 (9_OUT1C)
- net gp9: now also extra_gpio1.8 (Pin_8)
- net gp0: now reaches U1.2 (0_RX1_CRX2_CS1)
- net gp0: now also extra_gpio1.1 (Pin_1)
- net gp14: now reaches U1.21 (14_A0_TX3_SPDIF_OUT)
- net gp14: now also extra_gpio1.9 (Pin_9)
- net gp15: now reaches U1.22 (15_A1_RX3_SPDIF_IN)
- net gp15: now also extra_gpio1.10 (Pin_10)
- net I2C1_SCL: now reaches U1.23 (16_A2_RX4_SCL1)
- net I2C1_SCL: now also J4.4 (Pin_4), R15.1, STEMMA_QT_I2C1.4 (Pin_4)
- net I2C1_SDA: now reaches U1.24 (17_A3_TX4_SDA1)
- net I2C1_SDA: now also J4.3 (Pin_3), R14.2, STEMMA_QT_I2C1.3 (Pin_3)
- net I2C0_SDA: now reaches U1.25 (18_A4_SDA0)
- net I2C0_SCL: now reaches U1.26 (19_A5_SCL0)
- net gp22: now reaches U1.29 (22_A8_CTX1)
- net gp22: now also extra_gpio1.11 (Pin_11)
- net gp1: now reaches U1.3 (1_TX1_CTX2_MISO1)
- net gp1: now also extra_gpio1.2 (Pin_2)
- net gp23: now reaches U1.30 (23_A9_CRX1_MCLK1)
- net gp23: now also extra_gpio1.12 (Pin_12)
- net gp2: now reaches U1.4 (2_OUT2)
- net gp2: now also extra_gpio1.3 (Pin_3)
- net gp3: now reaches U1.5 (3_LRCLK2)
- net gp3: now also extra_gpio1.4 (Pin_4)
- net gp4: now reaches U1.6 (4_BCLK2)
- net gp4: now also extra_gpio1.5 (Pin_5)
- net gp6: now reaches U1.8 (6_OUT1D)
- net gp6: now also extra_gpio1.6 (Pin_6)
- new net: AGND_BRIDGE2.2 (B), C24.1
- new net audio_out_chan2: J1.3 (Pin_3), J2.R, JP6.2 (C)
- new net haptic_input: C24.2
- no-connect marks 1 -> 26
Other:
- added sheet drv2605_haptic_voice (drv2605_haptic_voice.kicad_sch)
- note added: "2.5mm pins"
- note added: "By default, only channel 1 (left channel) is used for output. But you can cut traces to change this. But then you have to cut the trace for the haptic chip"
- note added: "DRV2605 haptic chip"
- note added: "Hyaline Haptic Audio Player by Mads Kjeldgaard 2025"
- note added: "OUTPUT"
- note added: "TODO: - Buttons / UI? - Volume pot?"
- note added: "stemmaqt / i2c1"
- note removed: "Out jack"
- note removed: "Out pins"
- note removed: "power LED"
- moved on the sheet: J1, J2
